Commit message: Rotated and modified EE Xacro and URDFs

File: baxter_description/urdf/baxter_electric_gripper.urdf.xacro (robot description, xacro)
@@ -1,7 +1,14 @@
 <?xml version="1.0"?>
-<robot xmlns:xacro="http://www.ros.org/wiki/xacro" name="baxter_with_rethink_electric_gripper">
-  <xacro:include filename="$(find baxter_description)/urdf/baxter_base.xacro" />
+<robot xmlns:xacro="http://www.ros.org/wiki/xacro" name="baxter">
+  <xacro:include filename="$(find baxter_description)/urdf/baxter.urdf" />
   <xacro:include filename="$(find baxter_description)/urdf/rethink_electric_gripper.xacro" />
-  <xacro:rethink_electric_gripper side="right" gripper_side="r"/>
-  <xacro:rethink_electric_gripper side="left"  gripper_side="l"/>
+  <!-- Finger mesh index -->
+  <!--mesh filename="package://baxter_description/meshes/electric_gripper/fingers/00017816.DAE" /--> <!--basic_hard_tip-->
+  <!--mesh filename="package://baxter_description/meshes/electric_gripper/fingers/00030515.DAE" /--> <!--extended_wide -->
+  <!--mesh filename="package://baxter_description/meshes/electric_gripper/fingers/00030516.DAE" /--> <!-- standard_wide -->
+  <!--mesh filename="package://baxter_description/meshes/electric_gripper/fingers/00030517.DAE" /--> <!-- standard_narrow -->
+  <!--mesh filename="package://baxter_description/meshes/electric_gripper/fingers/00030518.DAE" /--> <!--extended_narrow /-->
+  <!--mesh filename="package://baxter_description/meshes/electric_gripper/fingers/00030535.DAE" /--> <!-- limiter -->
+  <xacro:rethink_electric_gripper side="right" gripper_side="r" finger_mesh="package://baxter_description/meshes/electric_gripper/fingers/extended_rotated.DAE"/>
+  <xacro:rethink_electric_gripper side="left"  gripper_side="l" finger_mesh="package://baxter_description/meshes/electric_gripper/fingers/extended_rotated.DAE"/>
 </robot>

File: baxter_description/urdf/rethink_electric_gripper.xacro (robot description, xacro)
@@ -1,10 +1,11 @@
 <?xml version="1.0"?>
 <robot xmlns:xacro="http://www.ros.org/wiki/xacro" name="rethink_electric_gripper">
-  <xacro:macro name="rethink_electric_gripper" params="side gripper_side">
+  <xacro:macro name="rethink_electric_gripper" params="side gripper_side finger_mesh">
     <!-- Base of end effector -->
-    <link name="${side}_gripper_base">
+    <link name="${side}_electric_gripper_base">
       <gravity>0</gravity>
       <visual>
-        <origin rpy="-1.57079632679 3.1415 0" xyz="0.00 0.00 0.025"/>
+        <!-- origin rpy="-1.57079632679 3.1415 0" xyz="0.00 0.00 0.025"/-->
+        <origin rpy="-1.57079632679 3.1415 0" xyz="0 0 0"/>
         <geometry>
           <mesh filename="package://baxter_description/meshes/electric_gripper/electric_gripper_base.DAE"/>
@@ -26,45 +27,24 @@
       </inertial>
     </link>
-    <link name="${side}_gripper">
-      <gravity>0</gravity>
-      <visual>
-        <origin rpy="0 0 0" xyz="0 0 0"/>
-        <geometry>
-          <box size="0.01 0.01 0.01"/>
-        </geometry>
-        <material name="rblack">
-          <color rgba="0 0 0 1"/>
-        </material>
-      </visual>
-      <inertial>
-        <origin rpy="0 0 0" xyz="0.000000 0.000000 0.000000"/>
-        <mass value="0.0001"/>
-        <inertia ixx="1e-08" ixy="0" ixz="0" iyy="1e-08" iyz="0" izz="1e-08"/>
-      </inertial>
-    </link>
-    <!-- Finger mesh index -->
-    <!--mesh filename="package://baxter_description/meshes/electric_gripper/fingers/00017816.DAE" /--> <!--basic_hard_tip-->
-    <!--mesh filename="package://baxter_description/meshes/electric_gripper/fingers/00030515.DAE" /--> <!--extended_wide -->
-    <!--mesh filename="package://baxter_description/meshes/electric_gripper/fingers/00030516.DAE" /--> <!-- standard_wide -->
-    <!--mesh filename="package://baxter_description/meshes/electric_gripper/fingers/00030517.DAE" /--> <!-- standard_narrow -->
-    <!--mesh filename="package://baxter_description/meshes/electric_gripper/fingers/00030518.DAE" /--> <!--extended_narrow /-->
-    <!--mesh filename="package://baxter_description/meshes/electric_gripper/fingers/00030535.DAE" /--> <!-- limiter -->
     <!-- Right finger -->
     <link name="${side}_gripper_r_finger">
       <gravity>0</gravity>
       <visual>
-        <origin rpy="0 1.57079632679 0" xyz="0.007 -0.036 0.0135"/>
+        <!-- origin rpy="0 1.57079632679 0" xyz="0.007 -0.036 0.0135"/ -->
+        <origin rpy="0 0 1.57079632679" xyz="0 0 0"/>
         <geometry>
-          <mesh filename="package://baxter_description/meshes/electric_gripper/fingers/extended_narrow.DAE" /> <!-- Long left finger-->
+          <mesh filename="${finger_mesh}" />
         </geometry>
       </visual>
       <collision>
-        <origin rpy="0 1.57079632679 0" xyz="0.007 -0.036 0.0135"/>
+        <!-- origin rpy="0 1.57079632679 0" xyz="0.007 -0.036 0.0135"/ -->
+        <origin rpy="0 0 1.57079632679" xyz="0 0 0"/>
         <geometry>
-          <mesh filename="package://baxter_description/meshes/electric_gripper/fingers/extended_narrow.DAE" /> <!-- Long left finger-->
+          <mesh filename="${finger_mesh}" />
         </geometry>
       </collision>
       <inertial>
-        <origin rpy="0 1.57079632679 0" xyz="0.007 -0.036 0.0135"/>
+        <!-- origin rpy="0 1.57079632679 0" xyz="0.007 -0.036 0.0135"/ -->
+        <origin rpy="0 0 1.57079632679" xyz="0 0 0"/>
         <!-- <mass value="0.00094542"/> -->
         <!-- <inertia ixx="2e-08" ixy="0" ixz="0" iyy="3e-08" iyz="0" izz="2e-08"/> -->
@@ -77,17 +57,20 @@
       <gravity>0</gravity>
       <visual>
-        <origin rpy="0 -1.57079632679 0" xyz="0.007 -0.036 -0.0135"/>
+        <!-- origin rpy="0 -1.57079632679 0" xyz="0.007 -0.036 -0.0135"/ -->
+        <origin rpy="0 0 -1.57079632679" xyz="0 0 0"/>
         <geometry>
-          <mesh filename="package://baxter_description/meshes/electric_gripper/fingers/extended_narrow.DAE" />
+          <mesh filename="${finger_mesh}" />
         </geometry>
       </visual>
       <collision>
-        <origin rpy="0 -1.57079632679 0" xyz="0.007 -0.036 -0.0135"/>
+        <!-- origin rpy="0 -1.57079632679 0" xyz="0.007 -0.036 -0.0135"/ -->
+        <origin rpy="0 0.0 -1.57079632679" xyz="0 0 0"/>
         <geometry>
-          <mesh filename="package://baxter_description/meshes/electric_gripper/fingers/extended_narrow.DAE" /> <!-- Long left finger-->
+          <mesh filename="${finger_mesh}" />
         </geometry>
       </collision>
       <inertial>
-        <origin rpy="0 -1.57079632679 0" xyz="0.007 -0.036 -0.0135"/>
+        <!-- origin rpy="0 -1.57079632679 0" xyz="0.007 -0.036 -0.0135"/ -->
+        <origin rpy="0 0 -1.57079632679" xyz="0 0 0"/>
         <!-- <mass value="0.00094542"/> -->
         <!-- <inertia ixx="2e-08" ixy="0" ixz="0" iyy="3e-08" iyz="0" izz="2e-08"/> -->
@@ -96,13 +79,14 @@
       </inertial>
     </link>
-    <!-- Base of Right end effector -->
-    <joint name="${side}_endpoint" type="fixed">
-      <origin rpy="1.57      0 0" xyz="-0.005 0.0 0.02"/>
-      <parent link="${side}_hand"/>
-      <child link="${side}_gripper"/>
+    <!-- Electric Gripper Base -->
+    <joint name="${gripper_side}_electric_gripper_base_joint" type="fixed">
+      <origin rpy="0 0 0" xyz="0 0 0.025"/>
+      <parent link="${side}_gripper_base"/>
+      <child link="${side}_electric_gripper_base"/>
     </joint>
     <!-- Right finger -->
     <joint name="${gripper_side}_gripper_r_finger_joint" type="prismatic">
-      <origin rpy="0 0 0" xyz="0.0 0.06 -0.035"/>
+      <!--origin rpy="1.57079632679 0 0" xyz="0.0 0.06 0.035"/-->
+      <origin rpy="0 0 0" xyz="0.0 0.035 0"/>
       <axis xyz="0 0 1"/>
       <parent link="${side}_gripper"/>
@@ -113,5 +97,6 @@
     <!-- Left finger -->
     <joint name="${gripper_side}_gripper_l_finger_joint" type="prismatic">
-      <origin rpy="0 0 0" xyz="0.0 0.06 0.035"/>
+      <!--origin rpy="1.57079632679 0 0" xyz="0.0 0.06 0.035"/-->
+      <origin rpy="0 0 0" xyz="0 -0.035 0"/>
       <axis xyz="0 0 1"/>
       <parent link="${side}_gripper"/>

Commit message: Added input paramters to rethink_electric_gripper.xacro

File: baxter_description/urdf/baxter_electric_gripper.urdf.xacro (robot description, xacro)
@@ -10,5 +10,5 @@
   <!--mesh filename="package://baxter_description/meshes/electric_gripper/fingers/00030518.DAE" /--> <!--extended_narrow /-->
   <!--mesh filename="package://baxter_description/meshes/electric_gripper/fingers/00030535.DAE" /--> <!-- limiter -->
-  <xacro:rethink_electric_gripper side="right" gripper_side="r" finger_mesh="package://baxter_description/meshes/electric_gripper/fingers/extended_rotated.DAE"/>
-  <xacro:rethink_electric_gripper side="left"  gripper_side="l" finger_mesh="package://baxter_description/meshes/electric_gripper/fingers/extended_rotated.DAE"/>
+  <xacro:rethink_electric_gripper side="right" gripper_side="r" finger_mesh="package://baxter_description/meshes/electric_gripper/fingers/extended_rotated.DAE" finger_mass="0.01" fingers_inverted="1" hole_number="1"/>
+  <xacro:rethink_electric_gripper side="left"  gripper_side="l" finger_mesh="package://baxter_description/meshes/electric_gripper/fingers/extended_rotated.DAE" finger_mass="0.01" fingers_inverted="1" hole_number="1"/>
 </robot>

File: baxter_description/urdf/rethink_electric_gripper.xacro (robot description, xacro)
@@ -1,11 +1,11 @@
 <?xml version="1.0"?>
 <robot xmlns:xacro="http://www.ros.org/wiki/xacro" name="rethink_electric_gripper">
-  <xacro:macro name="rethink_electric_gripper" params="side gripper_side finger_mesh">
+  <xacro:property name="pi" value="3.1415926535897931" />
+  <xacro:macro name="rethink_electric_gripper" params=" side gripper_side finger_mesh hole_number fingers_inverted finger_mass">
     <!-- Base of end effector -->
-    <link name="${side}_electric_gripper_base">
+    <link name="${side}_gripper_electric_base">
       <gravity>0</gravity>
       <visual>
-        <!-- origin rpy="-1.57079632679 3.1415 0" xyz="0.00 0.00 0.025"/-->
-        <origin rpy="-1.57079632679 3.1415 0" xyz="0 0 0"/>
+        <origin rpy="${-pi/2} ${pi} 0" xyz="0 0 0"/>
         <geometry>
           <mesh filename="package://baxter_description/meshes/electric_gripper/electric_gripper_base.DAE"/>
@@ -13,7 +13,7 @@
       </visual>
       <collision>
-        <origin rpy="0 0 0" xyz="0.007 0.007 0"/>
+        <origin rpy="${-pi/2} ${pi}  0" xyz="0.0 0.0 0"/>
         <geometry>
-          <cylinder length="0.1" radius="0.0275"/>
+          <cylinder length="0.1" radius="0.029"/>
         </geometry>
         <material name="darkred">
@@ -22,5 +22,5 @@
       </collision>
       <inertial>
-        <origin rpy="0 0 0" xyz="0.000000 0.000000 0.000000"/>
+        <origin rpy="${-pi/2} ${pi} 0" xyz="0.000000 0.000000 0.000000"/>
         <mass value="0.00094542"/>
         <inertia ixx="2e-08" ixy="0" ixz="0" iyy="3e-08" iyz="0" izz="2e-08"/>
@@ -31,6 +31,5 @@
       <gravity>0</gravity>
       <visual>
-        <!-- origin rpy="0 1.57079632679 0" xyz="0.007 -0.036 0.0135"/ -->
-        <origin rpy="0 0 1.57079632679" xyz="0 0 0"/>
+        <origin rpy="0 0 ${fingers_inverted*pi + pi/2}" xyz="0 0 0"/>
         <geometry>
           <mesh filename="${finger_mesh}" />
@@ -38,6 +37,5 @@
       </visual>
       <collision>
-        <!-- origin rpy="0 1.57079632679 0" xyz="0.007 -0.036 0.0135"/ -->
-        <origin rpy="0 0 1.57079632679" xyz="0 0 0"/>
+        <origin rpy="0 0 ${fingers_inverted*pi + pi/2}" xyz="0 0 0"/>
         <geometry>
           <mesh filename="${finger_mesh}" />
@@ -45,9 +43,6 @@
       </collision>
       <inertial>
-        <!-- origin rpy="0 1.57079632679 0" xyz="0.007 -0.036 0.0135"/ -->
-        <origin rpy="0 0 1.57079632679" xyz="0 0 0"/>
-        <!-- <mass value="0.00094542"/> -->
-        <!-- <inertia ixx="2e-08" ixy="0" ixz="0" iyy="3e-08" iyz="0" izz="2e-08"/> -->
-        <mass value="0.01"/>
+        <origin rpy="0 0 ${fingers_inverted*pi + pi/2}" xyz="0 0 0"/>
+        <mass value="${finger_mass}"/>
         <inertia ixx="0.01" ixy="0" ixz="0" iyy="0.01" iyz="0" izz="0.01"/>
       </inertial>
@@ -57,6 +52,5 @@
       <gravity>0</gravity>
       <visual>
-        <!-- origin rpy="0 -1.57079632679 0" xyz="0.007 -0.036 -0.0135"/ -->
-        <origin rpy="0 0 -1.57079632679" xyz="0 0 0"/>
+        <origin rpy="0 0 ${fingers_inverted*pi - pi/2}" xyz="0 0 0"/>
         <geometry>
           <mesh filename="${finger_mesh}" />
@@ -64,6 +58,5 @@
       </visual>
       <collision>
-        <!-- origin rpy="0 -1.57079632679 0" xyz="0.007 -0.036 -0.0135"/ -->
-        <origin rpy="0 0.0 -1.57079632679" xyz="0 0 0"/>
+        <origin rpy="0 0 ${fingers_inverted*pi - pi/2}" xyz="0 0 0"/>
         <geometry>
           <mesh filename="${finger_mesh}" />
@@ -71,38 +64,33 @@
       </collision>
       <inertial>
-        <!-- origin rpy="0 -1.57079632679 0" xyz="0.007 -0.036 -0.0135"/ -->
-        <origin rpy="0 0 -1.57079632679" xyz="0 0 0"/>
-        <!-- <mass value="0.00094542"/> -->
-        <!-- <inertia ixx="2e-08" ixy="0" ixz="0" iyy="3e-08" iyz="0" izz="2e-08"/> -->
-        <mass value="0.01"/>
+        <origin rpy="0 0 ${fingers_inverted*pi - pi/2}" xyz="0 0 0"/>
+        <mass value="${finger_mass}"/>
         <inertia ixx="0.01" ixy="0" ixz="0" iyy="0.01" iyz="0" izz="0.01"/>
       </inertial>
     </link>
     <!-- Electric Gripper Base -->
-    <joint name="${gripper_side}_electric_gripper_base_joint" type="fixed">
+    <joint name="${gripper_side}_gripper_electric_base_joint" type="fixed">
       <origin rpy="0 0 0" xyz="0 0 0.025"/>
       <parent link="${side}_gripper_base"/>
-      <child link="${side}_electric_gripper_base"/>
+      <child link="${side}_gripper_electric_base"/>
+    </joint>
+    <!-- Left finger -->
+    <joint name="${gripper_side}_gripper_l_finger_joint" type="prismatic">
+      <origin rpy="0 0 0" xyz="0 -0.0125 0.02"/>
+      <axis xyz="0 1 0"/>
+      <parent link="${side}_gripper_electric_base"/>
+      <child link="${side}_gripper_l_finger"/>
+      <limit effort="20.0" lower="-0.0125" upper="0.0095" velocity="5.0"/> <!-- mimic joint for lower is open -->
+      <dynamics damping="0.7" friction="0.0"/>
     </joint>
     <!-- Right finger -->
     <joint name="${gripper_side}_gripper_r_finger_joint" type="prismatic">
-      <!--origin rpy="1.57079632679 0 0" xyz="0.0 0.06 0.035"/-->
-      <origin rpy="0 0 0" xyz="0.0 0.035 0"/>
-      <axis xyz="0 0 1"/>
-      <parent link="${side}_gripper"/>
+      <origin rpy="0 0 0" xyz="0.0 0.0095 0.02"/>
+      <axis xyz="0 1 0"/>
+      <parent link="${side}_gripper_electric_base"/>
       <child link="${side}_gripper_r_finger"/>
-      <limit effort="20.0" lower="-0.0095" upper="0.0215" velocity="5.0"/> <!-- upper is open -->
+      <limit effort="20.0" lower="-0.0125" upper="0.0095" velocity="5.0"/> <!-- upper is open -->
       <dynamics damping="0.7" friction="0.0"/>
-    </joint>
-    <!-- Left finger -->
-    <joint name="${gripper_side}_gripper_l_finger_joint" type="prismatic">
-      <!--origin rpy="1.57079632679 0 0" xyz="0.0 0.06 0.035"/-->
-      <origin rpy="0 0 0" xyz="0 -0.035 0"/>
-      <axis xyz="0 0 1"/>
-      <parent link="${side}_gripper"/>
-      <child link="${side}_gripper_l_finger"/>
-      <limit effort="20.0" lower="-0.0215" upper="0.0095" velocity="5.0"/> <!-- mimic joint for lower is open -->
-      <dynamics damping="0.7" friction="0.0"/>
-      <mimic joint="${gripper_side}_gripper_r_finger_joint" offset="0"
+      <mimic joint="${gripper_side}_gripper_l_finger_joint" offset="0"
              multiplier="-1" />
     </joint>
