Commit message: Added Xacro Infra for Dynamic Grippers Constructs
- Rotated the long_narrow finger dae (for testing, will delete in future)
- Rotated and translated the paddle_tip dae so that the origin
  corresponds with the finger's tip. This should be standard for all
  finger tips in the future
- Added new xacro files corresponding to fingers and tips of fingers.
  Every new finger and tip will get its own xacro. This allows us to
  control the mass, rotation, and translation between different fingers
- Improved the baxter_electric_gripper.xacro to ask for intuitive
  descriptions of the electric gripper, such as finger mount points,
  finger and finger tip
- Removed the dependance on baxter.urdf.xacro - our base URDF will
  always be baxter.urdf to preserve backwards compatibility

File: baxter_description/urdf/baxter_electric_gripper.urdf.xacro (robot description, xacro)
@@ -3,12 +3,6 @@
   <xacro:include filename="$(find baxter_description)/urdf/baxter.urdf" />
   <xacro:include filename="$(find baxter_description)/urdf/rethink_electric_gripper.xacro" />
-  <!-- Finger mesh index -->
-  <!--mesh filename="package://baxter_description/meshes/electric_gripper/fingers/00017816.DAE" /--> <!--basic_hard_tip-->
-  <!--mesh filename="package://baxter_description/meshes/electric_gripper/fingers/00030515.DAE" /--> <!--extended_wide -->
-  <!--mesh filename="package://baxter_description/meshes/electric_gripper/fingers/00030516.DAE" /--> <!-- standard_wide -->
-  <!--mesh filename="package://baxter_description/meshes/electric_gripper/fingers/00030517.DAE" /--> <!-- standard_narrow -->
-  <!--mesh filename="package://baxter_description/meshes/electric_gripper/fingers/00030518.DAE" /--> <!--extended_narrow /-->
-  <!--mesh filename="package://baxter_description/meshes/electric_gripper/fingers/00030535.DAE" /--> <!-- limiter -->
-  <xacro:rethink_electric_gripper side="right" gripper_side="r" finger_mesh="package://baxter_description/meshes/electric_gripper/fingers/extended_rotated.DAE" finger_mass="0.01" fingers_inverted="1" hole_number="1"/>
-  <xacro:rethink_electric_gripper side="left"  gripper_side="l" finger_mesh="package://baxter_description/meshes/electric_gripper/fingers/extended_rotated.DAE" finger_mass="0.01" fingers_inverted="1" hole_number="1"/>
+  <xacro:rethink_electric_gripper side="left" gripper_side="l" l_finger="extended_narrow" l_finger_slot="1" add_l_finger_tip="true" l_finger_tip="paddle_tip" r_finger="extended_narrow" r_finger_slot="1" add_r_finger_tip="true" r_finger_tip="paddle_tip"/>
+  <xacro:rethink_electric_gripper side="right" gripper_side="r" l_finger="extended_narrow" l_finger_slot="1" add_l_finger_tip="false" l_finger_tip="false" r_finger="extended_narrow" r_finger_slot="1" add_r_finger_tip="false" r_finger_tip="false"/>
+  <!-- basic_hard_tip -->
 </robot>

File: baxter_description/urdf/rethink_electric_gripper.xacro (robot description, xacro)
@@ -2,5 +2,5 @@
 <robot xmlns:xacro="http://www.ros.org/wiki/xacro" name="rethink_electric_gripper">
   <xacro:property name="pi" value="3.1415926535897931" />
-  <xacro:macro name="rethink_electric_gripper" params=" side gripper_side finger_mesh hole_number fingers_inverted finger_mass">
+  <xacro:macro name="rethink_electric_gripper" params="side gripper_side  r_finger r_finger_slot add_r_finger_tip r_finger_tip l_finger l_finger_slot add_l_finger_tip l_finger_tip">
     <!-- Base of end effector -->
     <link name="${side}_gripper_electric_base">
@@ -13,5 +13,5 @@
       </visual>
       <collision>
-        <origin rpy="${-pi/2} ${pi}  0" xyz="0.0 0.0 0"/>
+        <origin rpy="${-pi/2} ${pi} 0" xyz="0.0 0.0 0"/>
         <geometry>
           <cylinder length="0.1" radius="0.029"/>
@@ -22,51 +22,15 @@
       </collision>
       <inertial>
-        <origin rpy="${-pi/2} ${pi} 0" xyz="0.000000 0.000000 0.000000"/>
-        <mass value="0.00094542"/>
+        <origin rpy="${-pi/2} ${pi} 0" xyz="0.0 0.0 0.0"/>
+        <mass value="0.3"/>
         <inertia ixx="2e-08" ixy="0" ixz="0" iyy="3e-08" iyz="0" izz="2e-08"/>
       </inertial>
     </link>
-    <!-- Right finger -->
-    <link name="${side}_gripper_r_finger">
-      <gravity>0</gravity>
-      <visual>
-        <origin rpy="0 0 ${fingers_inverted*pi + pi/2}" xyz="0 0 0"/>
-        <geometry>
-          <mesh filename="${finger_mesh}" />
-        </geometry>
-      </visual>
-      <collision>
-        <origin rpy="0 0 ${fingers_inverted*pi + pi/2}" xyz="0 0 0"/>
-        <geometry>
-          <mesh filename="${finger_mesh}" />
-        </geometry>
-      </collision>
-      <inertial>
-        <origin rpy="0 0 ${fingers_inverted*pi + pi/2}" xyz="0 0 0"/>
-        <mass value="${finger_mass}"/>
-        <inertia ixx="0.01" ixy="0" ixz="0" iyy="0.01" iyz="0" izz="0.01"/>
-      </inertial>
-    </link>
-    <!-- Left finger -->
-    <link name="${side}_gripper_l_finger">
-      <gravity>0</gravity>
-      <visual>
-        <origin rpy="0 0 ${fingers_inverted*pi - pi/2}" xyz="0 0 0"/>
-        <geometry>
-          <mesh filename="${finger_mesh}" />
-        </geometry>
-      </visual>
-      <collision>
-        <origin rpy="0 0 ${fingers_inverted*pi - pi/2}" xyz="0 0 0"/>
-        <geometry>
-          <mesh filename="${finger_mesh}" />
-        </geometry>
-      </collision>
-      <inertial>
-        <origin rpy="0 0 ${fingers_inverted*pi - pi/2}" xyz="0 0 0"/>
-        <mass value="${finger_mass}"/>
-        <inertia ixx="0.01" ixy="0" ixz="0" iyy="0.01" iyz="0" izz="0.01"/>
-      </inertial>
-    </link>
+    <!-- Left finger link -->
+    <xacro:include filename="$(find baxter_description)/urdf/${l_finger}.xacro" />
+    <xacro:finger_xacro gripper_side="${side}" finger_side="l" reflect="1" finger_tip="${l_finger_tip}" add_finger_tip="${add_l_finger_tip}"/>
+    <!-- Right finger link -->
+    <xacro:include filename="$(find baxter_description)/urdf/${r_finger}.xacro" />
+    <xacro:finger_xacro gripper_side="${side}" finger_side="r" reflect="-1" finger_tip="${r_finger_tip}" add_finger_tip="${add_r_finger_tip}"/>
     <!-- Electric Gripper Base -->
     <joint name="${gripper_side}_gripper_electric_base_joint" type="fixed">
@@ -77,21 +41,19 @@
     <!-- Left finger -->
     <joint name="${gripper_side}_gripper_l_finger_joint" type="prismatic">
-      <origin rpy="0 0 0" xyz="0 -0.0125 0.02"/>
+      <origin rpy="0 0 0" xyz="-0.0032 ${(l_finger_slot-1)*0.0095} 0.017"/>
       <axis xyz="0 1 0"/>
       <parent link="${side}_gripper_electric_base"/>
       <child link="${side}_gripper_l_finger"/>
-      <limit effort="20.0" lower="-0.0125" upper="0.0095" velocity="5.0"/> <!-- mimic joint for lower is open -->
+      <limit effort="20.0" lower="${(l_finger_slot-1)*0.0095 + 0.020833}" upper="${(l_finger_slot-1)*0.0095}" velocity="5.0"/>
       <dynamics damping="0.7" friction="0.0"/>
     </joint>
     <!-- Right finger -->
     <joint name="${gripper_side}_gripper_r_finger_joint" type="prismatic">
-      <origin rpy="0 0 0" xyz="0.0 0.0095 0.02"/>
+      <origin rpy="0 0 0" xyz="0.0 ${(r_finger_slot-1)*-0.0095} 0.017"/>
       <axis xyz="0 1 0"/>
       <parent link="${side}_gripper_electric_base"/>
       <child link="${side}_gripper_r_finger"/>
-      <limit effort="20.0" lower="-0.0125" upper="0.0095" velocity="5.0"/> <!-- upper is open -->
+      <limit effort="20.0" lower="${(r_finger_slot-1)*-0.0095 - 0.020833}" upper="${(r_finger_slot-1)*-0.0095}" velocity="5.0"/>
       <dynamics damping="0.7" friction="0.0"/>
-      <mimic joint="${gripper_side}_gripper_l_finger_joint" offset="0"
-             multiplier="-1" />
     </joint>
     <transmission name="gripper_${side}1">
